File: stm32f4-dev-module/stm32f4-dev-module.kicad_sch (KiCad schematic)
At the start: 20 parts, among them J1 SW, P1 USB_C_Plug, SW1 SW_SPST, SW2 SW_SPDT, U1 STM32F405RGT6, U2 USBLC6-2SC6, Y1 25MHz

Commit message: commit
Parts:
- added C12: 4u7, symbol Device:C_Polarized_Small
- added C13, C16: 100n, symbol Device:C_Small
- added C14, C15, C17: 1u, symbol Device:C_Small
- added D1: RED, symbol Device:LED
- added J2: Screw_Terminal_CAN, symbol Connector:Screw_Terminal_01x02
- added R2: 1k, symbol Device:R_Small
- added R3: 10k, symbol Device:R_Small
- added U3: SN65HVD230, Package_SO:SOIC-8_3.9x4.9mm_P1.27mm, symbol Interface_CAN_LIN:SN65HVD230
- added U4: AP2112K-3.3, Connector_USB:USB_C_Plug_Molex_105444, symbol Regulator_Linear:AP2112K-3.3
Connections:
- net +3.3V: now also J1.4 (Pin_4), C15.1, C16.1, C17.1, R2.1, U3.3 (VCC), U4.5 (VOUT)
- net CAN1_Rx: now also U3.4 (R)
- net CAN1_Tx: now also U3.1 (D)
- net GND: now also J1.1 (Pin_1), C12.2, C13.2, C14.2, C15.2, C16.2, C17.2, D1.1 (K), R3.2, U3.2 (GND), U4.2 (GND)
- net SWCLK: now also J1.2 (Pin_2)
- net SWDIO: now also J1.3 (Pin_3)
- net VBUS: now reaches P1.A4 (VBUS), P1.A9 (VBUS), P1.B4 (VBUS), P1.B9 (VBUS), U2.5 (VBUS)
- net VBUS: now also C12.1, C13.1, C14.1, U4.1 (VIN), U4.3 (EN)
- new net: J2.1 (Pin_1), U3.7 (CANH)
- new net: J2.2 (Pin_2), U3.6 (CANL)
- new net: D1.2 (A), R2.2
- new net: R3.1, U3.8 (Rs)
- no-connect marks 11 -> 12
Other:
- moved on the sheet: U2

Commit message: commmit
Parts:
- added C18: 100n, symbol Device:C_Small
- added C19: 2u2, symbol Device:C_Small
- added C20: 10n, symbol Device:C_Small
- added J3: I2C1, symbol Connector:Conn_01x04_Pin
- added J4: SPI1, Connector_PinHeader_1.00mm:PinHeader_2x03_P1.00mm_Vertical, symbol Connector_Generic:Conn_02x03_Top_Bottom
- added U5: ICM-42670-P, symbol eggsacc:ICM-42670-P
Connections:
- net +3.3V: now also C18.1, C19.1, C20.1, J3.4 (Pin_4), J4.4 (Pin_4), U5.5 (VDDIO), U5.8 (VDD)
- net GND: now also C18.2, C19.2, C20.2, J3.1 (Pin_1), J4.6 (Pin_6), U5.6 (GND), U5.7 (FSYNC)
- net I2C1_SCL: now also J3.2 (Pin_2)
- net I2C1_SDA: now also J3.3 (Pin_3)
- net ACCEL_INT: now reaches U1.16 (PA2)
- net ACCEL_INT: now also U5.4 (INT1/INT)
- net ACCEL_CS: now reaches U1.17 (PA3)
- net ACCEL_CS: now also U5.12 (AP_CS)
- net SPI1_CS: now reaches U1.20 (PA4)
- net SPI1_CS: now also J4.3 (Pin_3)
- net SPI1_CLK: now reaches U1.21 (PA5)
- net SPI1_CLK: now also J4.2 (Pin_2), U5.13 (AP_SCL/AP_SCLK)
- net SPI1_MISO: now reaches U1.22 (PA6)
- net SPI1_MISO: now also J4.1 (Pin_1), U5.1 (AP_SDO/AP_AD0)
- net SPI1_MOSI: now reaches U1.23 (PA7)
- net SPI1_MOSI: now also J4.5 (Pin_5), U5.14 (AP_SDA/AP_SDIO/AP_SDI)
- no-connect marks 12 -> 17
Other:
- moved on the sheet: C10, C11, Y1

Commit message: commit
Parts:
- added C21: 10n, symbol Device:C_Small
- added R4, R5: 60, symbol Device:R_Small
- added SW3: SW_DPST, symbol Switch:SW_DPST
Connections:
- net GND: now also C21.2
- net CANH: now reaches J2.1 (Pin_1), U3.7 (CANH)
- net CANH: now also R5.2
- net CANL: now reaches J2.2 (Pin_2), U3.6 (CANL)
- net CANL: now also R4.2
- new net: R5.1, SW3.1
- new net: C21.1, SW3.2, SW3.4
- new net: R4.1, SW3.3
Other:
- moved on the sheet: C14, C15, C16, C17, D1, J2, R2, R3, U3, U4
